File: Hardware/SmartWatch_System.brd (EAGLE design)
At the start: 46 x 35 mm, 105 parts, among them IC1 BQ25180YBGR, IC2 DRV2605YZFR, IC3 BMA421, IC9 RT6160AWSC, J1 503480-2400, J2 TC2030-IDC, J4 KH-TYPE-C-16P, Q1 20V/4.2A/52mΩ/1.4W, Q3 SI1308EDL-T1-GE3, SW1 2025-10-22_07-23-44_LIBRARY_E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

Commit message: Add files via upload
Parts:
- C14, C24, C37, C38, C39: device InkTime_v5:ESP32_C6_LIBRARY_1_ESP32_WROVER_EAGLE-LTSPICE_C0402 -> InkTime_v5:PERFECT_0402_0402
- C23: device rcl:HPC0201 -> InkTime_v5:GRM011R60J152KE01L_2_CAPC0201X13N
- C34, C42: device InkTime_v5:GRM011R60J152KE01L_1_0201 -> InkTime_v5:NORDIC_NRF_3_RESC0201_L
- C5: device rcl:HPC0201 -> InkTime_v5:NORDIC_NRF_3_RESC0201_L
- R2, R4: device rcl:R0201 -> InkTime_v5:ERA-1AEB3401C_0201
- R9: value 10K -> 10k
- moved C14 1.97 mm to (47.7, 76.1), turned to 180 degrees
- moved C39 1.53 mm to (41.7, 86.2), turned to 90 degrees
- moved C23 0.65 mm to (42.5, 88.3), turned to 270 degrees
- moved C24 0.61 mm to (42.2, 84.0), turned to 180 degrees
- moved C38 0.38 mm to (43.0, 81.8)
- moved R4 0.32 mm to (47.2, 76.9), turned to 0 degrees
- moved R9 0.26 mm to (47.6, 85.5)
- moved C37 0.16 mm to (46.7, 86.3)
- moved R2 0.16 mm to (45.8, 81.9)
- moved C5 0.08 mm to (50.8, 87.2)
Connections:
- net GND: now also C23.2, C24.2; no longer C23.1, C24.1
- net N$2: now also R4.2; no longer R4.1
- net N$3: now also R2.2; no longer R2.1
- net SCL/2.4C: now also R4.1; no longer R4.2
- net SDA/2.4C: now also R2.1; no longer R2.2
- net VREG: now also C23.1, C24.1; no longer C23.2, C24.2
Routing:
- net VBUS/2.6D: track 50.9 -> 51.9 mm
- net VBAT/1.2A: track 9.32 -> 10.0 mm
- net 3V3/2.4A: track 101.7 -> 102.3 mm
- net SDA/2.4C: track 23.7 -> 24.2 mm
Other:
- board text added: "3V3"
- board text added: "GND"
- board text added: "RST"
- board text added: "SCL"
- board text added: "SDA"
- board text added: "SWDCLK"
- board text added: "SWDIO"
- board text added: "SWO"
- board text added: "VBAT"
- board text added: "VREG"
