File: Hardware/SmartWatch_System.sch (EAGLE design)
At the start: 105 parts, among them IC1 BQ25180YBGR, IC2 DRV2605YZFR, IC3 BMA421, IC9 RT6160AWSC, J1 503480-2400, J2 TC2030-IDC, J4 KH-TYPE-C-16P, Q1 20V/4.2A/52mΩ/1.4W, Q3 SI1308EDL-T1-GE3, SW1 2025-10-22_07-23-44_LIBRARY_E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

Commit message: Add files via upload
Parts:
- C14, C24, C37, C38, C39: device InkTime_v5:ESP32_C6_LIBRARY_1_ESP32_WROVER_EAGLE-LTSPICE_CC0402 -> InkTime_v5:PERFECT_0402_CAP_0402
- C23: device rcl:C-EUHPC0201 -> InkTime_v5:GRM011R60J152KE01L_2_GRM011R60J152KE01L
- C5: device rcl:C-EUHPC0201 -> InkTime_v5:NORDIC_NRF_3_CAPACITOR_0201_L
- R2, R4: device rcl:R-EU_R0201 -> InkTime_v5:ERA-1AEB3401C_CPF0201D7K68C1
- R9: value 10K -> 10k
Connections:
- net GND: now also C23.2, C24.2; no longer C23.1, C24.1
- net N$2: now also R4.2; no longer R4.1
- net N$3: now also R2.2; no longer R2.1
- net SCL/2.4C: now also R4.1; no longer R4.2
- net SDA/2.4C: now also R2.1; no longer R2.2
- net VREG: now also C23.1, C24.1; no longer C23.2, C24.2
Other:
- moved on the sheet: C23, C24
